Commit message: Fix precision profile compatibility and saturate teleop joint targets

File: assets/SO101/urdf/so101_isaaclab.urdf (robot description, URDF)
Before this commit: robot so101_calibrated, 8 links, 7 joints
Joints:
- joint elbow_flex: limit lower=-1.74533 upper=1.5708 effort=10 velocity=10 -> lower=-1.8325964625997164 upper=1.6580664625997164 effort=10 velocity=10
- joint shoulder_lift: limit lower=-1.74533 upper=1.74533 effort=10 velocity=10 -> lower=-1.8325964625997164 upper=1.8325964625997164 effort=10 velocity=10
- joint shoulder_pan: limit lower=-1.91986 upper=1.91986 effort=10 velocity=10 -> lower=-2.0071264625997163 upper=2.0071264625997163 effort=10 velocity=10
- joint wrist_flex: limit lower=-1.65806 upper=1.65806 effort=10 velocity=10 -> lower=-1.7453264625997165 upper=1.7453264625997165 effort=10 velocity=10
